File: PCB_Rev1/Main_Board_Rev1/_autosave-cstar-power.kicad_sch (KiCad schematic)
At the start: 49 parts, among them IC1 LT8648SEV#PBF, J4 Conn_01x02_Pin, J5 XT60PW-M, J6 Conn_01x02_Pin, J7 Conn_01x02_Pin, J8 Conn_01x02_Pin, U1 AZ1117IH-3.3TRG1

Commit message: LDO component files imported
Other:
- note added: "Buck Converter 2: 12V to 5V, 3A"
- note removed: "Buck Converter 1: 12V to 5V, 3A"
Changed lines of the file:
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@@
 		)
 	)
-	(text "Buck Converter 1: 12V to 5V, 3A\n"
+	(text "Buck Converter 2: 12V to 5V, 3A\n"
 		(exclude_from_sim no)
 		(at 43.18 191.77 0)
