File: PCB_Rev1/Main_Board_Rev1/cstar-lidar.kicad_sch (KiCad schematic)
At the start: 1 part, among them J3 532610771

Commit message: Update cstar-lidar.kicad_sch
Parts:
- J3: footprint CSTAR-MainBoard-Footprints:MOLEX_532610771 -> Connector_Molex:Molex_PicoBlade_53261-0771_1x07-1MP_P1.25mm_Horizontal
Changed lines of the file:
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@@
 			)
 		)
-		(property "Footprint" "CSTAR-MainBoard-Footprints:MOLEX_532610771"
+		(property "Footprint" "Connector_Molex:Molex_PicoBlade_53261-0771_1x07-1MP_P1.25mm_Horizontal"
 			(at 172.72 95.25 0)
 			(effects
