File: PCB_Rev1/Main_Board_Rev1/cstar-lidar.kicad_sch (KiCad schematic)
At the start: 1 part, among them J11 532610771

Commit message: LCSC + CSV changes
Parts:
- J11: LCSC (none) -> C505276
Changed lines of the file:
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@@
+			)
+		)
+		(property "LCSC" "C505276"
+			(at 172.72 95.25 0)
+			(effects
+				(font
+					(size 1.27 1.27)
+				)
+				(hide yes)
 			)
 		)
