File: PCB_Rev1/Main_Board_Rev1/cstar-io.kicad_sch (KiCad schematic)
At the start: 11 parts, among them J2 Conn_01x04_Socket, J3 691137710002, Q1 AO3400A, Q2 AO3400A, Q3 AO3400A, Q4 IRFHM9331TRPBF

Commit message: final touches... not rlly
Parts:
- Q4: footprint Footprints:POWER_FET_3.0 -> Footprints:NEW_power_FET
Changed lines of the file:
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@@
 			)
 		)
-		(property "Footprint" "Footprints:POWER_FET_3.0"
+		(property "Footprint" "Footprints:NEW_power_FET"
 			(at 219.075 63.5 0)
 			(effects

Commit message: GND net to M5 holes
Parts:
- Q4: footprint Footprints:NEW_power_FET -> Footprints:POWER_FET_3.0
Changed lines of the file:
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@@
 			)
 		)
-		(property "Footprint" "Footprints:NEW_power_FET"
+		(property "Footprint" "Footprints:POWER_FET_3.0"
 			(at 219.075 63.5 0)
 			(effects
