File: PCB_Rev1/Mic_Board_Omni_New/Omni_New/Omni_New.kicad_pcb (KiCad board)
At the start: 2 copper layers, 51 x 31.5 mm, 30 parts, among them J1 Conn_01x03_Pin, J2 532610771, J3 S2B-ZR-SM4A-TF_LF__SN_, U1 OPA1671IDBVR

Commit message: New
Parts:
- removed J3: S2B-ZR-SM4A-TF_LF__SN_, Footprints:Mic_Conn
Routing:
- net GND: track 144.3 -> 126.3 mm
