File: PCB_Rev1/Mic_Board_Omni_New/Mic_Board_Omni_New/Mic_Board_Omni_New.kicad_sch (KiCad schematic)
At the start: 30 parts, among them J1 Conn_01x03_Pin, J2 532610771, U1 OPA1671IDBVR

Commit message: New omni created
Parts:
- removed J1: Conn_01x03_Pin, Connector_PinHeader_2.54mm:PinHeader_1x03_P2.54mm_Vertical, symbol Connector:Conn_01x03_Pin
- removed MK1: Microphone, symbol Device:Microphone
- added J3: S2B-ZR-SM4A-TF_LF__SN_, Footprints:Mic_Conn, symbol Mic Connectors:S2B-ZR-SM4A-TF_LF__SN_
- added R8, R9: 10k, Resistor_SMD:R_0805_2012Metric, symbol Device:R_Small_US
- R7: value 1k -> 18k
Connections:
- net +3V3: now also J2.6, R8.2; no longer J2.5
- net GND: now also J2.7, J3.2, J3.S1 (SHIELD), J3.S2 (SHIELD__1), R9.1; no longer J2.6
- net at J2.1: now also U2.10 (LRCK); no longer U2.9 (SDTO)
- net at J2.2: now also U2.12 (BICK); no longer U2.10 (LRCK)
- net at U2.11 (MCLK): now also R9.2; no longer J2.3
- net at J2.4: no longer U2.12 (BICK)
- net at U2.13 (PDN): now also R8.1
- net at U2.15 (FSEL): now also J2.3
- net at C2.1, R2.2: now also J3.1
- new net: J2.5, U2.9 (SDTO)
- no-connect marks 1 -> 2
Other:
- moved on the sheet: J2, R7
